File: PCB/board.brd (EAGLE design)
At the start: 79 x 60 mm, 32 parts, among them IC1 MEGA1284P-SQUARE, IC2 MC33269D-3.3, J1 DCJ0202, Q1 CRYSTAL_16MHZ_SMD, Q2 BUZ10, U1 OPA564AIDWD

Commit message: Michael and Matthew, Silkscreening done
Parts:
- SCK_LED: value RED -> BLUE
- renumbered LED1 to 5V_LED, LED2 to SCK_LED, LED3 to 3V3_LED
Connections:
- net N$10 renamed 13
- net N$11 renamed 12
- net N$12 renamed 11
- net N$13 renamed 10
- net N$14 renamed 9
- net N$15 renamed 26
- net N$16 renamed 25
- net N$17 renamed 24
- net N$18 renamed 23
- net N$19 renamed 22
- net N$20 renamed 21
- net N$25 renamed 35
- net N$26 renamed 34
- net N$27 renamed 33
- net N$28 renamed 32
- net N$29 renamed 31
- net N$30 renamed 30
- net N$31 renamed 40
- net N$32 renamed 41
- net N$33 renamed 42
- net N$35 renamed 44
- net N$8 renamed 15
- net N$9 renamed 14
Other:
- board text added: "+"
- board text added: "+ -"
- board text added: "+ Heater"
- board text added: "- Heater"
- board text added: "10"
- board text added: "11"
- board text added: "12"
- board text added: "13"
- board text added: "14"
- board text added: "15"
- board text added: "21"
- board text added: "22"
- board text added: "23"
- board text added: "24"
- board text added: "25"
- board text added: "26"
- board text added: "30"
- board text added: "31"
- board text added: "32"
- board text added: "33"
- board text added: "34"
- board text added: "35"
- board text added: "40"
- board text added: "41"
- board text added: "42"
- board text added: "44"
- board text added: "5V"
- board text added: "9"
- board text added: "Designed by: Nipun Dasanayaka Michael Manceor Brandon Nikpreljevic Matthew Stachowiak Jacob Weisberg"
- board text added: "GND"
- board text added: "Heater Connector"
- board text added: "IFLAG (36)"
- board text added: "MISO"
- board text added: "MOSI"
- board text added: "Modular Temperature Control Board"
- board text added: "Peltier Connector"
- board text added: "RESET"
- board text added: "Reset"
- board text added: "SCK"
- board text added: "SCL"
- board text added: "SDA"
- board text added: "TFLAG (37)"

Commit message: Finalized Board #1
Parts:
- added JP1: (no value), pinhead:1X02
- added PIN_15_LED: BLUE, led:CHIP-LED0603
- added R7: 150, rcl:R0603
- moved C4 60.3 mm to (66.0, 33.1)
- moved C3 40.4 mm to (47.9, 36.1), turned to 90 degrees
- moved C5 18.2 mm to (46.8, 32.4)
- moved C6 15.8 mm to (40.4, 34.2), turned to 270 degrees
- moved Q1 13.9 mm to (43.6, 33.4), turned to 180 degrees
Connections:
- removed net +HEATER: HEATER_CONNECTOR.1
- new net N$1: PIN_15_LED.A, R7.1
- net +12V: now also HEATER_CONNECTOR.1
- net +3V3: now also JP1.1
- net 15: now also R7.2
- net GND: now also JP1.2, PIN_15_LED.C
Routing:
- net N$2: track 64.5 -> 2.55 mm, vias 2 -> 0
- net +12V: track 44.5 -> 79.7 mm
- net N$4: track 31.0 -> 12.3 mm, vias 2 -> 0
- net N$3: track 27.1 -> 9.39 mm, vias 2 -> 0
- net +5V: track 110.3 -> 125.8 mm
- net +3V3: track 20.7 -> 33.6 mm
- net GND: track 16.0 -> 23.2 mm, vias 2 -> 4
- net PELTIER_5V: track 39.6 -> 34.7 mm
- net 15: track 23.0 -> 27.6 mm
- net N$1: track 0.00 -> 2.84 mm
- net IFLAG: track 69.1 -> 70.9 mm
Other:
- board text added: "+3V3"
